Commit message: fix(vehicle.xacro): fix position of mesh model
Signed-off-by: Ryohsuke Mitsudome <ryohsuke.mitsudome@tier4.jp>

File: edgar_vehicle_description/urdf/vehicle.xacro (robot description, xacro)
@@ -6,5 +6,5 @@
   <link name="base_link">
     <visual>
-      <origin xyz="${vehicle_info['/**']['ros__parameters']['wheel_base']/2.0} 0 0" rpy="0 0 0"/>
+      <origin xyz="0 0 0" rpy="0 0 0"/>
       <geometry>
         <mesh filename="package://edgar_vehicle_description/mesh/edgar.dae" scale="1 1 1"/>
